Commit message: feat: camera rotation controller, slam map loader, waypoint corrections

File: robot_urdf/urdf/robot6.xacro (robot description, xacro)
@@ -117,13 +117,13 @@
   <link name="camera_link">
 	    <collision>
-	      <origin xyz="0 0 0.025" rpy="0 0 0"/>
+	      <origin xyz="0 0 0.3" rpy="0 0 0"/>
 	      <geometry>
-		<box size="0.05 0.05 0.05"/>
+		<box size="0.05 0.05 0.1"/>
 	      </geometry>
 	    </collision>
 	    <visual>
-	      <origin xyz="0 0 0.025" rpy="0 0 0"/>
+	      <origin xyz="0 0 0.05" rpy="0 0 0"/>
 	      <geometry>
-		<box size="0.05 0.05 0.05"/>
+		<box size="0.05 0.05 0.1"/>
 	      </geometry>
 	      <material name="red">
@@ -137,10 +137,10 @@
 	    </inertial>
   </link>
-  <joint name="camera_joint" type="fixed">
-	    <axis xyz="0 1 0" />
-	    <origin xyz="0.23 0 0.0" rpy="0 0 0"/>
+  <joint name="camera_joint" type="continuous">
+	    <axis xyz="0 0 1" />
+	    <origin xyz="0.23 0 0.2" rpy="0 0 0"/>
 	    <parent link="link_chassis"/>
 	    <child link="camera_link"/>
-    </joint>
+  </joint>
   <link name="laser_link">
 	    <collision>
@@ -171,3 +171,27 @@
 	    <child link="laser_link"/>
 	 </joint>
+   <transmission name="camera_trans">
+  <type>transmission_interface/SimpleTransmission</type>
+  <joint name="camera_joint">
+    <hardwareInterface>hardware_interface/VelocityJointInterface</hardwareInterface>
+  </joint>
+  <actuator name="camera_motor">
+    <mechanicalReduction>m1</mechanicalReduction>
+  </actuator>
+</transmission>
+  <!-- ros2_control tag -->
+  <ros2_control name="my_robot_control" type="system">
+    <hardware>
+      <plugin>gazebo_ros2_control/GazeboSystem</plugin>
+    </hardware>
+    <joint name="camera_joint">
+      <command_interface name="velocity">
+        <param name="min">-10</param>
+        <param name="max">10</param>
+      </command_interface>
+      <state_interface name="position"/>
+      <state_interface name="velocity"/>
+      <state_interface name="effort"/>
+    </joint>
+  </ros2_control>
 </robot>
